File: RESONANSE_FLC/PCB/STM32_BOARD/LCSDR.kicad_pcb (KiCad board)
At the start: 2 copper layers, 100 x 95 mm, 135 parts, among them J1 F, J10 Conn_01x01, J11 Conn_01x01, J12 USB_B_Mini, J2 IDC10 Serial Wire, J3 LC/G3UUR, J4 Conn_01x04, J5 Jack-DC, J6 NEO-7M, J7 Conn_01x01, J8 Conn_01x01, J9 Conn_01x01, K1 TIANBO-HJR-4102-L, K2 TIANBO-HJR-4102-L, K3 TIANBO-HJR-4102-L, K4 TIANBO-HJR-4102-L, Q1 MMBT2222, Q10 SS9018, Q11 SS9018, Q12 SS9018, Q2 MMBT2222, Q3 MMBT2222, Q4 MMBT2222, Q5 BFT92, Q6 BFT92, Q7 BC817, Q8 BC857, Q9 BF998, SW1 SW_Push_Dual, SW2 SW_Push_Dual, SW3 SW_Push_Dual, SW4 SW_Push_Dual, SW5 ENCODER, SW6 SW_Push_Dual, U15 Nokia_5110_LCD, U2 FM24CL16B, U3 STM32F401RCTx, U4 AP1117-33, U5 MC34063, Y1 20Mhz, Y2 Crystal

Commit message: PIC PCB
Parts:
- removed C5, C6: 100nF, UI:C_1206_0603
- removed D5: LL4148, Diodes_SMD:D_MiniMELF_Handsoldering
- removed K1, K2: TIANBO-HJR-4102-L, Relays_ThroughHole:Relay_SPDT_HJR-4102
- removed Q3: MMBT2222, TO_SOT_Packages_SMD:SOT-23_Handsoldering
- removed R3: 2.7k, Resistors_THT:R_Axial_DIN0204_L3.6mm_D1.6mm_P7.62mm_Horizontal
- added C43: 100nF, UI:C_1206_0603, B.Cu at (154.2, 55.5)
- added C48: 100nF, UI:C_1206_0603, B.Cu at (148.5, 61.2)
- added C49: 100nF, UI:C_1206_0603, B.Cu at (135.4, 66.8)
- added D9: BAV99, TO_SOT_Packages_SMD:SOT-23, B.Cu at (132.7, 62.2)
- added Q13: BC847, TO_SOT_Packages_SMD:SOT-23, B.Cu at (125.8, 69.4)
- added R32: 10k, UI:R_1206_0603, B.Cu at (138.4, 66.3)
- added R33: 4.7k, UI:R_1206_0603, B.Cu at (138.7, 60.4)
- added R34: 220, UI:R_1206_0603, B.Cu at (142.3, 61.5)
- added R35: 4.7k, UI:R_1206_0603, B.Cu at (128.0, 73.5)
- added R36: 220, UI:R_1206_0603, B.Cu at (133.6, 72.3)
- D4: value LL4148 -> BAV99; footprint Diodes_SMD:D_MiniMELF_Handsoldering -> TO_SOT_Packages_SMD:SOT-23
- D6: footprint Diodes_SMD:D_MiniMELF_Handsoldering -> Diodes_SMD:D_MiniMELF
- D7, D8, Q11, Q12, Q5, Q6, Q8: footprint TO_SOT_Packages_SMD:SOT-23_Handsoldering -> TO_SOT_Packages_SMD:SOT-23
- Q10: value SS9018 -> SS9018(J8); footprint TO_SOT_Packages_SMD:SOT-23_Handsoldering -> TO_SOT_Packages_SMD:SOT-23
- Q2: value MMBT2222 -> BC847; footprint TO_SOT_Packages_SMD:SOT-23_Handsoldering -> TO_SOT_Packages_SMD:SOT-23
- Q4: value MMBT2222 -> MMBT2222LT1G; footprint TO_SOT_Packages_SMD:SOT-23_Handsoldering -> TO_SOT_Packages_SMD:SOT-23
- Q9: footprint TO_SOT_Packages_SMD:SOT-143_Handsoldering -> TO_SOT_Packages_SMD:SOT-143
- R10: value 56R -> 4.7k
- R12: value 2.7k -> 4.7k
- R17, R5: footprint Resistors_ThroughHole:R_Axial_DIN0204_L3.6mm_D1.6mm_P1.90mm_Vertical -> UI:R_1206_0603
- R2: value 2.7k -> 10k; footprint Resistors_THT:R_Axial_DIN0204_L3.6mm_D1.6mm_P7.62mm_Horizontal -> UI:R_1206_0603
- R22: value 47k -> 36k; footprint Resistors_ThroughHole:R_Axial_DIN0204_L3.6mm_D1.6mm_P7.62mm_Horizontal -> UI:R_1206_0603
- R23: footprint Resistors_THT:R_Axial_DIN0204_L3.6mm_D1.6mm_P7.62mm_Horizontal -> UI:R_1206_0603
- moved Q9 54.4 mm to (95.5, 52.6)
- moved C19 54.0 mm to (102.1, 53.1), turned to 180 degrees
- moved R20 52.1 mm to (95.8, 47.2), turned to 180 degrees
- moved R18 51.0 mm to (102.1, 50.5), turned to 180 degrees
- moved C21 50.1 mm to (89.6, 50.0), turned to 270 degrees
- moved D7 48.6 mm to (99.2, 57.8), turned to 90 degrees
- moved R22 48.1 mm to (88.3, 54.2)
- moved C20 45.8 mm to (107.5, 50.5), turned to 180 degrees
- moved R17 45.5 mm to (105.7, 56.3), turned to 180 degrees
- moved Q10 44.9 mm to (88.1, 57.8)
- moved C15 43.7 mm to (111.2, 56.3), turned to 180 degrees
- moved C16 42.8 mm to (111.2, 59.1), turned to 180 degrees
- moved L4 42.5 mm to (147.1, 46.8), turned to 0 degrees
- moved D8 36.3 mm to (112.6, 50.5), turned to 180 degrees
- moved R2 34.7 mm to (144.6, 57.8), turned to 0 degrees
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Connections:
- C14 pad 2: GND -> Net-(C14-Pad2)
- C3 pad 1: REL_1 -> Net-(C3-Pad1)
- D4 pad 1: +12V -> Net-(C48-Pad2)
- D4 pad 2: REL_1 -> Net-(C3-Pad1)
- J12 pad 1: Net-(J12-Pad1) -> (no net)
- J12 pad 4: Net-(J12-Pad4) -> (no net)
- J2 pad 7: Net-(J2-Pad7) -> (no net)
- J2 pad 8: Net-(J2-Pad8) -> (no net)
- K3 pad 12: Net-(K1-Pad12) -> Net-(C14-Pad1)
- K3 pad 7: Net-(K3-Pad7) -> (no net)
- L4 pad 1: Net-(K1-Pad6) -> Net-(C14-Pad1)
- L4 pad 2: GND -> Net-(C43-Pad2)
- Q10 pad 1: GND -> Net-(C21-Pad2)
- Q10 pad 2: Net-(C21-Pad2) -> GND
- Q2 pad 1: GND -> Net-(Q2-Pad1)
- Q2 pad 2: Net-(C4-Pad1) -> GND
- Q2 pad 3: REL_1 -> Net-(C3-Pad1)
- Q4 pad 1: GND -> Net-(C8-Pad1)
- Q4 pad 2: Net-(C8-Pad1) -> GND
- Q5 pad 1: Net-(K1-Pad12) -> Net-(C14-Pad1)
- Q6 pad 3: Net-(K1-Pad12) -> Net-(C14-Pad1)
- R2 pad 1: Net-(C4-Pad1) -> +12V
- R2 pad 2: REL_1_MCU -> Net-(C3-Pad1)
- U2 pad 1: Net-(U2-Pad1) -> (no net)
- U2 pad 2: Net-(U2-Pad2) -> (no net)
- U2 pad 3: Net-(U2-Pad3) -> (no net)
- U3 pad 22: Net-(U3-Pad22) -> (no net)
- U3 pad 23: Net-(U3-Pad23) -> (no net)
- U3 pad 24: Net-(U3-Pad24) -> (no net)
- U3 pad 25: Net-(U3-Pad25) -> (no net)
- U3 pad 26: Net-(U3-Pad26) -> (no net)
- U3 pad 27: Net-(U3-Pad27) -> (no net)
- U3 pad 28: Net-(U3-Pad28) -> (no net)
- U3 pad 29: Net-(U3-Pad29) -> (no net)
- U3 pad 33: I2S_LRCK -> (no net)
- U3 pad 34: I2S_SCLK -> (no net)
- U3 pad 4: Net-(U3-Pad4) -> (no net)
- U3 pad 42: Net-(U3-Pad42) -> (no net)
- U3 pad 43: Net-(U3-Pad43) -> (no net)
- U3 pad 57: Net-(U3-Pad57) -> (no net)
- U3 pad 58: Net-(U3-Pad58) -> (no net)
- U3 pad 59: Net-(U3-Pad59) -> (no net)
- U3 pad 61: Net-(U3-Pad61) -> (no net)
- U3 pad 62: Net-(U3-Pad62) -> (no net)
- U3 pad 8: BAND0 -> (no net)
Routing:
- net GND: track 697.2 -> 187.0 mm, vias 172 -> 49
- net +12V: track 320.1 -> 151.6 mm
- net +3V3: track 312.2 -> 214.2 mm
- net F_LC: track 57.9 -> 0.00 mm
- net MCU_RESET: track 50.7 -> 0.00 mm, vias 2 -> 0
- net F_Q: track 60.6 -> 11.4 mm
- net Net-(K1-Pad12): track 46.0 -> 0.00 mm, vias 1 -> 0
- net SWO: track 44.6 -> 0.00 mm, vias 2 -> 0
- net SWCLK: track 38.5 -> 0.00 mm
- net REL_0: track 28.7 -> 0.00 mm
- net REL_1: track 26.3 -> 0.00 mm
- net Net-(C46-Pad1): track 24.7 -> 0.40 mm
- net Net-(C20-Pad2): track 22.3 -> 0.00 mm
- net Net-(C17-Pad2): track 21.6 -> 0.00 mm
- net Net-(J2-Pad10): track 15.6 -> 0.00 mm
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Other:
- outline, holes or cut-outs redrawn
